File: slave.sch (EAGLE design)
At the start: 209 parts, among them J1 PHOENIX_1778641, J2 EB21A-06-D, J3 EB21A-06-D, J4 EB21A-06-D, J5 EB21A-06-D, Q1 DMN2056U-7, Q10 DMN2056U-7, Q11 DMN2056U-7, Q12 DMN2056U-7, Q13 DMN2056U-7, Q14 DMN2056U-7, Q15 DMN2056U-7, Q16 DMN2056U-7, Q17 DMN2056U-7, Q18 DMN2056U-7, Q19 DMN2056U-7, Q2 DMN2056U-7, Q20 DMN2056U-7, Q21 DMN2056U-7, Q3 DMN2056U-7, Q4 DMN2056U-7, Q5 DMN2056U-7, Q6 DMG2301L-7, Q7 DMN2056U-7, Q8 DMN2056U-7, Q9 DMN2056U-7, U1 ESP32-DEVKIT-V1, U2 AP2112K-3.3TRG1

Commit message: schematic finalized
Parts:
- removed J1: PHOENIX_1778641, ML_library:PHOENIX_1778641
- removed U1: ESP32-DEVKIT-V1, ESP32-DEVKIT-V1:ESP32-DEVKIT-V1
- added D25, D26, D27, D28, D29, D30, D31, D32, D33, D34, D35, D36, D37, D38, D39, D40, D41, D42, D43, D44, D45: VLMY1500-GS08, ML_library:VLMY1500-GS08
- added J6, J7, J8: 282837-9, 282837-9:282837-9
- added J9: 1715250000, 1715250000-2pin_screw_terminal_block:1715250000
- added Q22, Q23, Q24, Q25, Q26, Q27, Q28, Q29, Q30, Q31, Q32, Q33, Q34, Q35, Q36, Q37, Q38, Q39, Q40, Q41, Q42: DMN2056U-7, ML_library:DMN2056U-7SOT23
- added R100, R103, R106, R109, R112, R115, R118, R121, R124, R127, R130, R70, R73, R76, R79, R82, R85, R88, R91, R94, R97: 220, OPL_Resistor:SMD-RES-0R-1%-1/10W(0603)
- added R101, R104, R107, R110, R113, R116, R119, R122, R125, R128, R131, R71, R74, R77, R80, R83, R86, R89, R92, R95, R98: 150, OPL_Resistor:SMD-RES-1.2K-1%-1/10W(0603)
- added R102, R105, R108, R111, R114, R117, R120, R123, R126, R129, R132, R72, R75, R78, R81, R84, R87, R90, R93, R96, R99: 6.8k, OPL_Resistor:SMD-RES-0R-1%-1/10W(0603)
- added U$1, U$2: PPTC151LFBN-RC, PPTC151LFBN-RC:PPTC151LFBN-RC
- added U3, U4, U5: MCP23008-E/P, MCP23008-E_P:MCP23008-E/P
- added U6, U7, U8, U9: MC74HCT4851ADR2G, MC74HCT4851ADR2G:MC74HCT4851ADR2G
Connections:
- removed net N$11: U1.TX0
- removed net N$12: U1.RX2
- removed net N$13: U1.TX2
- removed net N$14: U1.D22
- removed net N$16: U1.D23
- removed net N$17: U1.D25
- removed net N$19: U1.D26
- removed net N$20: U1.D27
- removed net N$22: U1.D32
- removed net N$23: U1.D33
- removed net N$25: U1.D35
- removed net N$26: U1.D34
- removed net N$28: CB2.2, PR_CS4.VIOUT
- removed net N$30: CB4.2, PR_CS1.VIOUT
- removed net N$32: CB6.2, PR_CS2.VIOUT
- removed net N$34: CB8.2, PR_CS3.VIOUT
- removed net N$36: CB10.2, PR_CS5.VIOUT
- removed net N$38: CB12.2, PR_CS6.VIOUT
- removed net N$40: CB14.2, PR_CS7.VIOUT
- removed net N$42: CB16.2, PR_CS8.VIOUT
- removed net N$44: CB18.2, PR_CS9.VIOUT
- removed net N$46: CB20.2, PR_CS10.VIOUT
- removed net N$48: CB22.2, PR_CS11.VIOUT
- removed net N$50: CB24.2, PR_CS12.VIOUT
- removed net N$52: CB26.2, PR_CS13.VIOUT
- removed net N$54: CB28.2, PR_CS14.VIOUT
- removed net N$56: CB30.2, PR_CS15.VIOUT
- removed net N$58: CB32.2, PR_CS16.VIOUT
- removed net N$60: CB34.2, PR_CS17.VIOUT
- removed net N$62: CB36.2, PR_CS18.VIOUT
- removed net N$64: CB38.2, PR_CS19.VIOUT
- removed net N$66: CB40.2, PR_CS20.VIOUT
- removed net N$7 (its old number): J1.P$1, J1.P$2, RECT.2
- removed net N$81: U1.VIN
- removed net N$82: U1.EN
- removed net N$83: U1.VP
- removed net N$84: U1.VN
- removed net N$85: U1.D2
- removed net N$86: U1.D4
- removed net N$87: U1.D5
- removed net N$88: U1.D12
- removed net N$89: U1.D13
- removed net N$90: U1.D14
- removed net N$91: U1.D15
- removed net N$92: U1.D18
- removed net N$93: U1.D19
- removed net N$94: U1.D21
- new net +12V: J9.2, RECT.2
- new net CS_SEL0: U$2.P$6, U6.A, U7.A, U8.A, U9.A
- new net CS_SEL1: U$2.P$4, U6.B, U7.B, U8.B, U9.B
- new net CS_SEL2: U$2.P$3, U6.C, U7.C, U8.C, U9.C
- new net D0_A: R70.2, R71.2, U3.GP0
- new net D0_A+: J8.8, Q22.S
- new net D0_B: R73.2, R74.2, U3.GP1
- new net D0_B+: J8.7, Q23.S
- new net D0_C: R76.2, R77.2, U3.GP2
- new net D0_C+: J8.6, Q24.S
- new net D0_D: R79.2, R80.2, U3.GP3
- new net D0_D+: J8.5, Q25.S
- new net D0_E: R82.2, R83.2, U3.GP4
- new net D0_E+: J8.4, Q26.S
- new net D0_F: R100.2, R101.2, U3.GP5
- new net D0_F+: J8.3, Q32.S
- new net D0_G: R103.2, R104.2, U3.GP6
- new net D0_G+: J8.2, Q33.S
- new net D0_GND: R102.1, R105.1, R72.1, R75.1, R78.1, R81.1, R84.1
- new net D1_A: R85.2, R86.2, U4.GP0
- new net D1_A+: J6.8, Q27.S
- new net D1_B: R88.2, R89.2, U4.GP1
- new net D1_B+: J6.7, Q28.S
- new net D1_C: R91.2, R92.2, U4.GP2
- new net D1_C+: J6.6, Q29.S
- new net D1_D: R94.2, R95.2, U4.GP3
- new net D1_D+: J6.5, Q30.S
- new net D1_E: R97.2, R98.2, U4.GP4
- new net D1_E+: J6.4, Q31.S
- new net D1_F: R106.2, R107.2, U4.GP5
- new net D1_F+: J6.3, Q34.S
- new net D1_G: R109.2, R110.2, U4.GP6
- new net D1_G+: J6.2, Q35.S
- new net D1_GND: R108.1, R111.1, R87.1, R90.1, R93.1, R96.1, R99.1
- new net D23: U$2.P$1
- new net D2_A: R112.2, R113.2, U5.GP0
- new net D2_A+: J7.8, Q36.S
- new net D2_B: R115.2, R116.2, U5.GP1
- new net D2_B+: J7.7, Q37.S
- new net D2_C: R118.2, R119.2, U5.GP2
- new net D2_C+: J7.6, Q38.S
- new net D2_D: R121.2, R122.2, U5.GP3
- new net D2_D+: J7.5, Q39.S
- new net D2_E: R124.2, R125.2, U5.GP4
- new net D2_E+: J7.4, Q40.S
- new net D2_F: R127.2, R128.2, U5.GP5
- new net D2_F+: J7.3, Q41.S
- new net D2_G: R130.2, R131.2, U5.GP6
- new net D2_G+: J7.2, Q42.S
- new net D2_GND: R114.1, R117.1, R120.1, R123.1, R126.1, R129.1, R132.1
- new net I_OA: CB16.2, PR_CS8.VIOUT, U7.X1
- new net I_OGF: CB18.2, PR_CS9.VIOUT, U7.X2
- new net I_OGL: CB20.2, PR_CS10.VIOUT, U7.X3
- new net I_OGR: CB22.2, PR_CS11.VIOUT, U7.X4
- new net I_OR: CB14.2, PR_CS7.VIOUT, U7.X0
- new net I_PA: CB24.2, PR_CS12.VIOUT, U6.X1
- new net I_PGF: CB36.2, PR_CS18.VIOUT, U6.X2
- new net I_PGL: CB38.2, PR_CS19.VIOUT, U6.X3
- new net I_PGR: CB40.2, PR_CS20.VIOUT, U6.X4
- new net I_PR: CB12.2, PR_CS6.VIOUT, U6.X0
- new net I_SA: CB6.2, PR_CS2.VIOUT, U8.X1
- new net I_SGF: CB8.2, PR_CS3.VIOUT, U8.X2
- new net I_SGL: CB2.2, PR_CS4.VIOUT, U8.X3
- new net I_SGR: CB10.2, PR_CS5.VIOUT, U8.X4
- new net I_SPA: CB28.2, PR_CS14.VIOUT, U9.X1
- new net I_SPGF: CB30.2, PR_CS15.VIOUT, U9.X2
- new net I_SPGL: CB32.2, PR_CS16.VIOUT, U9.X3
- new net I_SPGR: CB34.2, PR_CS17.VIOUT, U9.X4
- new net I_SPR: CB26.2, PR_CS13.VIOUT, U9.X0
- new net I_SR: CB4.2, PR_CS1.VIOUT, U8.X0
- new net N$100: D31.2, R89.1
- new net N$101: D32.2, R92.1
- new net N$102: D33.2, R95.1
- new net N$103: D34.2, R98.1
- new net N$104: D35.2, R101.1
- new net N$105: D36.2, R104.1
- new net N$106: D37.2, R107.1
- new net N$107: D38.2, R110.1
- new net N$108: D39.2, R113.1
- new net N$109: D40.2, R116.1
- new net N$110: D41.2, R119.1
- new net N$111: D42.2, R122.1
- new net N$112: D43.2, R125.1
- new net N$113: D44.2, R128.1
- new net N$114: D45.2, R131.1
- new net N$80: D25.2, R71.1
- new net N$95: D26.2, R74.1
- new net N$96: D27.2, R77.1
- new net N$97: D28.2, R80.1
- new net N$98: D29.2, R83.1
- new net N$99: D30.2, R86.1
- new net O_CURRENT: U$1.P$5, U7.X
- new net P_CURRENT: U$1.P$7, U6.X
- new net Q1G20: Q22.G, R70.1, R72.2
- new net Q1G21: Q23.G, R73.1, R75.2
- new net Q1G22: Q24.G, R76.1, R78.2
- new net Q1G23: Q25.G, R79.1, R81.2
- new net Q1G24: Q26.G, R82.1, R84.2
- new net Q1G25: Q27.G, R85.1, R87.2
- new net Q1G26: Q28.G, R88.1, R90.2
- new net Q1G27: Q29.G, R91.1, R93.2
- new net Q1G28: Q30.G, R94.1, R96.2
- new net Q1G29: Q31.G, R97.1, R99.2
- new net Q1G30: Q32.G, R100.1, R102.2
- new net Q1G31: Q33.G, R103.1, R105.2
- new net Q1G32: Q34.G, R106.1, R108.2
- new net Q1G33: Q35.G, R109.1, R111.2
- new net Q1G34: Q36.G, R112.1, R114.2
- new net Q1G35: Q37.G, R115.1, R117.2
- new net Q1G36: Q38.G, R118.1, R120.2
- new net Q1G37: Q39.G, R121.1, R123.2
- new net Q1G38: Q40.G, R124.1, R126.2
- new net Q1G39: Q41.G, R127.1, R129.2
- new net Q1G40: Q42.G, R130.1, R132.2
- new net SCL: U$2.P$2, U3.SCL, U4.SCL, U5.SCL
- new net SDA: U$2.P$5, U3.SDA, U4.SDA, U5.SDA
- new net SP_CURRENT: U$1.P$4, U9.X
- new net S_CURRENT: U$1.P$6, U8.X
- new net VIN_ESP: U$1.P$15
- net +5V: now also U3.*RESET, U3.VDD, U4.*RESET, U4.A0, U4.VDD, U5.*RESET, U5.A1, U5.VDD, U6.VCC, U7.VCC, U8.VCC, U9.VCC
- net 3V3: now also U$2.P$15; no longer U1.3V3
- net EN: now also U$1.P$1
- net GND: now also J6.1, J7.1, J8.1, U$1.P$14, U$2.P$14, U3.A0, U3.A1, U3.A2, U3.VSS, U4.A1, U4.A2, U4.VSS, U5.A0, U5.A2, U5.VSS, U6.ENABLE, U6.GND, U6.X5, U6.X6, U6.X7, U7.ENABLE, U7.GND, U7.X5, U7.X6, U7.X7, U8.ENABLE, U8.GND, U8.X5, U8.X6, U8.X7, U9.ENABLE, U9.GND, U9.X5, U9.X6, U9.X7; no longer C2.1, COUT1.1, COUT2.1, COUT3.1, COUT4.1, Q1.S, Q10.S, Q11.S, Q12.S, Q13.S, Q14.S, Q15.S, Q16.S, Q17.S, Q18.S, Q19.S, Q2.S, Q20.S, Q21.S, Q3.S, Q4.S, Q5.S, Q7.S, Q8.S, Q9.S, R1.2, R10.1, R14.1, R18.1, R21.1, R25.1, R27.1, R30.1, R36.1, R39.1, R42.1, R45.1, R48.1, R51.1, R54.1, R57.1, R60.1, R63.1, R66.1, R69.1, R7.1, REG.AGND, REG.PGND, REG.PGND_2, REG.PGND_3, REG.PGND_4, U1.GND
- net JP2: now also D25.1, D26.1, D27.1, D28.1, D29.1, D30.1, D31.1, D32.1, D33.1, D34.1, D35.1, D36.1, D37.1, D38.1, D39.1, D40.1, D41.1, D42.1, D43.1, D44.1, D45.1
- net N$6: now also C2.1, COUT1.1, COUT2.1, COUT3.1, COUT4.1, R1.2, REG.AGND, REG.PGND, REG.PGND_2, REG.PGND_3, REG.PGND_4; no longer U1.RX0
- net N$9: now also J9.1; no longer J1.P$3, J1.P$4
- net OA+: now also Q13.S
- net OGF+: now also Q14.S
- net OGL+: now also Q15.S
- net OGR+: now also Q16.S
- net OLED_GND: now also R42.1, R45.1, R48.1, R51.1, R54.1; no longer PR_CS10.IP+, PR_CS11.IP+, PR_CS7.IP+, PR_CS8.IP+, PR_CS9.IP+
- net OR+: now also Q12.S
- net PA: now also U$1.P$12
- net PA+: now also Q2.S
- net PGF: now also U$1.P$11
- net PGF+: now also Q3.S
- net PGL: now also U$1.P$10
- net PGL+: now also Q4.S
- net PGR: now also U$1.P$9
- net PGR+: now also Q5.S
- net PLED_GND: now also R10.1, R14.1, R18.1, R25.1, R57.1, R60.1, R63.1, R66.1, R69.1, R7.1; no longer PR_CS12.IP+, PR_CS18.IP+, PR_CS19.IP+, PR_CS20.IP+, PR_CS6.IP+
- net PR: now also U$1.P$13
- net PR+: now also Q1.S
- net SA: now also U$1.P$3
- net SA+: now also Q8.S
- net SGF: now also U$1.P$2
- net SGF+: now also Q9.S
- net SGL: now also U$2.P$13
- net SGL+: now also Q10.S
- net SGR: now also U$2.P$12
- net SGR+: now also Q11.S
- net SLED_GND: now also R21.1, R27.1, R30.1, R36.1, R39.1; no longer PR_CS1.IP+, PR_CS2.IP+, PR_CS3.IP+, PR_CS4.IP+, PR_CS5.IP+
- net SPA: now also U$2.P$10
- net SPA+: now also Q18.S
- net SPGF: now also U$2.P$9
- net SPGF+: now also Q19.S
- net SPGL: now also U$2.P$8
- net SPGL+: now also Q20.S
- net SPGR: now also U$2.P$7
- net SPGR+: now also Q21.S
- net SPLED_GND: no longer PR_CS13.IP+, PR_CS14.IP+, PR_CS15.IP+, PR_CS16.IP+, PR_CS17.IP+
- net SPR: now also U$2.P$11
- net SPR+: now also Q17.S
- net SR: now also U$1.P$8
- net SR+: now also Q7.S
- net VIN: now also J6.9, J7.9, J8.9, PR_CS1.IP+, PR_CS10.IP+, PR_CS11.IP+, PR_CS12.IP+, PR_CS13.IP+, PR_CS14.IP+, PR_CS15.IP+, PR_CS16.IP+, PR_CS17.IP+, PR_CS18.IP+, PR_CS19.IP+, PR_CS2.IP+, PR_CS20.IP+, PR_CS3.IP+, PR_CS4.IP+, PR_CS5.IP+, PR_CS6.IP+, PR_CS7.IP+, PR_CS8.IP+, PR_CS9.IP+, Q22.D, Q23.D, Q24.D, Q25.D, Q26.D, Q27.D, Q28.D, Q29.D, Q30.D, Q31.D, Q32.D, Q33.D, Q34.D, Q35.D, Q36.D, Q37.D, Q38.D, Q39.D, Q40.D, Q41.D, Q42.D
Other:
- note added: "Overhead Lamp FETs and Port"
- note added: "Primary Lamp FETs and Port"
- note added: "Secondary Lamp FETs and Port"
- note added: "Spare Lamp FETs and Port"
- note added: "Timer Digit 0 FETs and Port"
- note added: "Timer Digit 1 FETs and Port"
- note added: "Timer Digit 2 FETs and Port"
- note removed: "LED ports"
- moved on the sheet: C2, C3, C4, C5, CB, CB1, CB10, CB11, CB12, CB13, CB14, CB15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

Commit message: removed backup files, finalized board layoout
Parts:
- removed D10, D8, D9: B5819W SL, ML_library:SCHOTTKY_SOD123
- removed PR_CS1, PR_CS10, PR_CS11, PR_CS12, PR_CS13, PR_CS14, PR_CS15, PR_CS16, PR_CS17, PR_CS18, PR_CS19, PR_CS2, PR_CS20, PR_CS3, PR_CS4, PR_CS5, PR_CS6, PR_CS7, PR_CS8, PR_CS9: ACS723LLCTR-10AU-T, ACS723LLCTR-10AU-T:ACS723LLCTR-10AU-T
- removed Q6: DMG2301L-7, ML_library:DMG2301L-7
- removed R32: 1k, OPL_Resistor:SMD-RES-1.5K-1%-1/16W(0402)
- removed R33: 10k, OPL_Resistor:SMD-RES-1.5K-1%-1/16W(0402)
- added OA_CS, OGF_CS, OGL_CS, OGR_CS, OR_CS, PA_CS, PGF_CS, PGL_CS, PGR_CS, PR_CS, SA_CS, SGF_CS, SGL_CS, SGR_CS, SPA_CS, SPGF_CS, SPGL_CS, SPGR_CS, SPR_CS, SR_CS: ACS723LLCTR-10AU-T, ACS723LLCTR-10AU-T:ACS723LLCTR-10AU-T
- renumbered U$1 to ESP_LEFT_HDR, U$2 to ESP_RIGHT_HDR
Connections:
- removed net 3V3_F: Q6.D
- removed net N$10: D8.C, D9.C, R32.1
- removed net N$35: CB9.1, PR_CS5.GND
- removed net N$47: CB21.1, PR_CS11.GND
- removed net N$5: D10.C, Q6.S
- removed net N$59: CB33.1, PR_CS17.GND
- removed net N$65: CB39.1, PR_CS20.GND
- removed net PMOS_G: Q6.G, R32.2, R33.2
- removed net VBAT: D9.A
- removed net VUSB: D8.A
- new net N$13: CB9.1, PGR_CS.GND
- new net N$14: CB21.1, SGR_CS.GND
- new net N$16: CB33.1, OGR_CS.GND
- new net N$17: CB39.1, SPGR_CS.GND
- net +5V: now also OA_CS.BW_SEL, OA_CS.VCC, OGF_CS.BW_SEL, OGF_CS.VCC, OGL_CS.BW_SEL, OGL_CS.VCC, OGR_CS.BW_SEL, OGR_CS.VCC, OR_CS.BW_SEL, OR_CS.VCC, PA_CS.BW_SEL, PA_CS.VCC, PGF_CS.BW_SEL, PGF_CS.VCC, PGL_CS.BW_SEL, PGL_CS.VCC, PGR_CS.BW_SEL, PGR_CS.VCC, PR_CS.BW_SEL, PR_CS.VCC, SA_CS.BW_SEL, SA_CS.VCC, SGF_CS.BW_SEL, SGF_CS.VCC, SGL_CS.BW_SEL, SGL_CS.VCC, SGR_CS.BW_SEL, SGR_CS.VCC, SPA_CS.BW_SEL, SPA_CS.VCC, SPGF_CS.BW_SEL, SPGF_CS.VCC, SPGL_CS.BW_SEL, SPGL_CS.VCC, SPGR_CS.BW_SEL, SPGR_CS.VCC, SPR_CS.BW_SEL, SPR_CS.VCC, SR_CS.BW_SEL, SR_CS.VCC; no longer PR_CS1.BW_SEL, PR_CS1.VCC, PR_CS10.BW_SEL, PR_CS10.VCC, PR_CS11.BW_SEL, PR_CS11.VCC, PR_CS12.BW_SEL, PR_CS12.VCC, PR_CS13.BW_SEL, PR_CS13.VCC, PR_CS14.BW_SEL, PR_CS14.VCC, PR_CS15.BW_SEL, PR_CS15.VCC, PR_CS16.BW_SEL, PR_CS16.VCC, PR_CS17.BW_SEL, PR_CS17.VCC, PR_CS18.BW_SEL, PR_CS18.VCC, PR_CS19.BW_SEL, PR_CS19.VCC, PR_CS2.BW_SEL, PR_CS2.VCC, PR_CS20.BW_SEL, PR_CS20.VCC, PR_CS3.BW_SEL, PR_CS3.VCC, PR_CS4.BW_SEL, PR_CS4.VCC, PR_CS5.BW_SEL, PR_CS5.VCC, PR_CS6.BW_SEL, PR_CS6.VCC, PR_CS7.BW_SEL, PR_CS7.VCC, PR_CS8.BW_SEL, PR_CS8.VCC, PR_CS9.BW_SEL, PR_CS9.VCC
- net 3V3: no longer D10.A
- net GND: no longer R33.1
- net I_OA: now also OA_CS.VIOUT; no longer PR_CS8.VIOUT
- net I_OGF: now also OGF_CS.VIOUT; no longer PR_CS9.VIOUT
- net I_OGL: now also OGL_CS.VIOUT; no longer PR_CS10.VIOUT
- net I_OGR: now also OGR_CS.VIOUT; no longer PR_CS11.VIOUT
- net I_OR: now also OR_CS.VIOUT; no longer PR_CS7.VIOUT
- net I_PA: now also PA_CS.VIOUT; no longer PR_CS12.VIOUT
- net I_PGF: now also PGF_CS.VIOUT; no longer PR_CS18.VIOUT
- net I_PGL: now also PGL_CS.VIOUT; no longer PR_CS19.VIOUT
- net I_PGR: now also PGR_CS.VIOUT; no longer PR_CS20.VIOUT
- net I_PR: now also PR_CS.VIOUT; no longer PR_CS6.VIOUT
- net I_SA: now also SA_CS.VIOUT; no longer PR_CS2.VIOUT
- net I_SGF: now also SGF_CS.VIOUT; no longer PR_CS3.VIOUT
- net I_SGL: now also SGL_CS.VIOUT; no longer PR_CS4.VIOUT
- net I_SGR: now also SGR_CS.VIOUT; no longer PR_CS5.VIOUT
- net I_SPA: now also SPA_CS.VIOUT; no longer PR_CS14.VIOUT
- net I_SPGF: now also SPGF_CS.VIOUT; no longer PR_CS15.VIOUT
- net I_SPGL: now also SPGL_CS.VIOUT; no longer PR_CS16.VIOUT
- net I_SPGR: now also SPGR_CS.VIOUT; no longer PR_CS17.VIOUT
- net I_SPR: now also SPR_CS.VIOUT; no longer PR_CS13.VIOUT
- net I_SR: now also SR_CS.VIOUT; no longer PR_CS1.VIOUT
- net N$29: now also SR_CS.GND; no longer PR_CS1.GND
- net N$31: now also SA_CS.GND; no longer PR_CS2.GND
- net N$33: now also SGF_CS.GND; no longer PR_CS3.GND
- net N$37: now also PR_CS.GND; no longer PR_CS6.GND
- net N$39: now also OR_CS.GND; no longer PR_CS7.GND
- net N$4: now also SGL_CS.GND; no longer PR_CS4.GND
- net N$41: now also OA_CS.GND; no longer PR_CS8.GND
- net N$43: now also OGF_CS.GND; no longer PR_CS9.GND
- net N$45: now also OGL_CS.GND; no longer PR_CS10.GND
- net N$49: now also PA_CS.GND; no longer PR_CS12.GND
- net N$51: now also SPR_CS.GND; no longer PR_CS13.GND
- net N$53: now also SPA_CS.GND; no longer PR_CS14.GND
- net N$55: now also SPGF_CS.GND; no longer PR_CS15.GND
- net N$57: now also SPGL_CS.GND; no longer PR_CS16.GND
- net N$61: now also PGF_CS.GND; no longer PR_CS18.GND
- net N$63: now also PGL_CS.GND; no longer PR_CS19.GND
- net OA_IP-: now also OA_CS.IP-; no longer PR_CS8.IP-
- net OGF_IP-: now also OGF_CS.IP-; no longer PR_CS9.IP-
- net OGL_IP-: now also OGL_CS.IP-; no longer PR_CS10.IP-
- net OGR_IP-: now also OGR_CS.IP-; no longer PR_CS11.IP-
- net OR_IP-: now also OR_CS.IP-; no longer PR_CS7.IP-
- net PA_IP-: now also PA_CS.IP-; no longer PR_CS12.IP-
- net PGF_IP-: now also PGF_CS.IP-; no longer PR_CS18.IP-
- net PGL_IP-: now also PGL_CS.IP-; no longer PR_CS19.IP-
- net PGR_IP-: now also PGR_CS.IP-; no longer PR_CS20.IP-
- net PR_IP-: now also PR_CS.IP-; no longer PR_CS6.IP-
- net SA_IP-: now also SA_CS.IP-; no longer PR_CS2.IP-
- net SGF_IP-: now also SGF_CS.IP-; no longer PR_CS3.IP-
- net SGL_IP-: now also SGL_CS.IP-; no longer PR_CS4.IP-
- net SGR_IP-: now also SGR_CS.IP-; no longer PR_CS5.IP-
- net SPA_IP-: now also SPA_CS.IP-; no longer PR_CS14.IP-
- net SPGF_IP-: now also SPGF_CS.IP-; no longer PR_CS15.IP-
- net SPGL_IP-: now also SPGL_CS.IP-; no longer PR_CS16.IP-
- net SPGR_IP-: now also SPGR_CS.IP-; no longer PR_CS17.IP-
- net SPR_IP-: now also SPR_CS.IP-; no longer PR_CS13.IP-
- net SR_IP-: now also SR_CS.IP-; no longer PR_CS1.IP-
- net VIN: now also OA_CS.IP+, OGF_CS.IP+, OGL_CS.IP+, OGR_CS.IP+, OR_CS.IP+, PA_CS.IP+, PGF_CS.IP+, PGL_CS.IP+, PGR_CS.IP+, PR_CS.IP+, SA_CS.IP+, SGF_CS.IP+, SGL_CS.IP+, SGR_CS.IP+, SPA_CS.IP+, SPGF_CS.IP+, SPGL_CS.IP+, SPGR_CS.IP+, SPR_CS.IP+, SR_CS.IP+; no longer PR_CS1.IP+, PR_CS10.IP+, PR_CS11.IP+, PR_CS12.IP+, PR_CS13.IP+, PR_CS14.IP+, PR_CS15.IP+, PR_CS16.IP+, PR_CS17.IP+, PR_CS18.IP+, PR_CS19.IP+, PR_CS2.IP+, PR_CS20.IP+, PR_CS3.IP+, PR_CS4.IP+, PR_CS5.IP+, PR_CS6.IP+, PR_CS7.IP+, PR_CS8.IP+, PR_CS9.IP+
Other:
- moved on the sheet: C2, C3, C4, C5, CB, CB1, CB10, CB11, CB12, CB13, CB14, CB15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

Commit message: changed header, but clearance issues
Parts:
- removed ESP_LEFT_HDR, ESP_RIGHT_HDR: PPTC151LFBN-RC, PPTC151LFBN-RC:PPTC151LFBN-RC
- added ESP_HDR_LEFT, ESP_HDR_RIGHT: PPTC191LFBN-RC, PPTC191LFBN-RC:PPTC191LFBN-RC
Connections:
- removed net D23: ESP_RIGHT_HDR.P$1
- removed net N$13: CB9.1, PGR_CS.GND
- removed net N$14: CB21.1, SGR_CS.GND
- removed net N$16: CB33.1, OGR_CS.GND
- removed net N$17: CB39.1, SPGR_CS.GND
- removed net N$29: CB3.1, SR_CS.GND
- removed net N$31: CB5.1, SA_CS.GND
- removed net N$33: CB7.1, SGF_CS.GND
- removed net N$37: CB11.1, PR_CS.GND
- removed net N$39: CB13.1, OR_CS.GND
- removed net N$4: CB1.1, SGL_CS.GND
- removed net N$41: CB15.1, OA_CS.GND
- removed net N$43: CB17.1, OGF_CS.GND
- removed net N$45: CB19.1, OGL_CS.GND
- removed net N$49: CB23.1, PA_CS.GND
- removed net N$51: CB25.1, SPR_CS.GND
- removed net N$53: CB27.1, SPA_CS.GND
- removed net N$55: CB29.1, SPGF_CS.GND
- removed net N$57: CB31.1, SPGL_CS.GND
- removed net N$61: CB35.1, PGF_CS.GND
- removed net N$63: CB37.1, PGL_CS.GND
- removed net VIN_ESP: ESP_LEFT_HDR.P$15
- new net 5V0: ESP_HDR_LEFT.1
- new net ESP_EN: ESP_HDR_LEFT.18
- new net GPIO1: ESP_HDR_RIGHT.16
- new net GPIO10: ESP_HDR_LEFT.3
- new net GPIO11: ESP_HDR_LEFT.2
- new net GPIO3: ESP_HDR_RIGHT.15
- new net GPIO6: ESP_HDR_RIGHT.1
- new net GPIO7: ESP_HDR_RIGHT.2
- new net GPIO8: ESP_HDR_RIGHT.3
- new net GPIO9: ESP_HDR_LEFT.4
- net 3V3: now also ESP_HDR_LEFT.19; no longer ESP_RIGHT_HDR.P$15
- net CS_SEL0: now also ESP_HDR_LEFT.5; no longer ESP_RIGHT_HDR.P$6
- net CS_SEL1: now also ESP_HDR_LEFT.7; no longer ESP_RIGHT_HDR.P$4
- net CS_SEL2: now also ESP_HDR_LEFT.8; no longer ESP_RIGHT_HDR.P$3
- net EN: no longer ESP_LEFT_HDR.P$1
- net GND: now also CB1.1, CB11.1, CB13.1, CB15.1, CB17.1, CB19.1, CB21.1, CB23.1, CB25.1, CB27.1, CB29.1, CB3.1, CB31.1, CB33.1, CB35.1, CB37.1, CB39.1, CB5.1, CB7.1, CB9.1, ESP_HDR_LEFT.6, ESP_HDR_RIGHT.13, ESP_HDR_RIGHT.19, OA_CS.GND, OGF_CS.GND, OGL_CS.GND, OGR_CS.GND, OR_CS.GND, PA_CS.GND, PGF_CS.GND, PGL_CS.GND, PGR_CS.GND, PR_CS.GND, SA_CS.GND, SGF_CS.GND, SGL_CS.GND, SGR_CS.GND, SPA_CS.GND, SPGF_CS.GND, SPGL_CS.GND, SPGR_CS.GND, SPR_CS.GND, SR_CS.GND; no longer ESP_LEFT_HDR.P$14, ESP_RIGHT_HDR.P$14
- net O_CURRENT: now also ESP_HDR_LEFT.16; no longer ESP_LEFT_HDR.P$5
- net PA: now also ESP_HDR_LEFT.10; no longer ESP_LEFT_HDR.P$12
- net PGF: now also ESP_HDR_LEFT.11; no longer ESP_LEFT_HDR.P$11
- net PGL: now also ESP_HDR_LEFT.12; no longer ESP_LEFT_HDR.P$10
- net PGR: now also ESP_HDR_LEFT.13; no longer ESP_LEFT_HDR.P$9
- net PR: now also ESP_HDR_LEFT.9; no longer ESP_LEFT_HDR.P$13
- net P_CURRENT: now also ESP_HDR_LEFT.14; no longer ESP_LEFT_HDR.P$7
- net SA: now also ESP_HDR_RIGHT.9; no longer ESP_LEFT_HDR.P$3
- net SCL: now also ESP_HDR_RIGHT.17; no longer ESP_RIGHT_HDR.P$2
- net SDA: now also ESP_HDR_RIGHT.14; no longer ESP_RIGHT_HDR.P$5
- net SGF: now also ESP_HDR_RIGHT.10; no longer ESP_LEFT_HDR.P$2
- net SGL: now also ESP_HDR_RIGHT.11; no longer ESP_RIGHT_HDR.P$13
- net SGR: now also ESP_HDR_RIGHT.12; no longer ESP_RIGHT_HDR.P$12
- net SPA: now also ESP_HDR_RIGHT.5; no longer ESP_RIGHT_HDR.P$10
- net SPGF: now also ESP_HDR_RIGHT.6; no longer ESP_RIGHT_HDR.P$9
- net SPGL: now also ESP_HDR_RIGHT.7; no longer ESP_RIGHT_HDR.P$8
- net SPGR: now also ESP_HDR_RIGHT.8; no longer ESP_RIGHT_HDR.P$7
- net SPR: now also ESP_HDR_RIGHT.4; no longer ESP_RIGHT_HDR.P$11
- net SP_CURRENT: now also ESP_HDR_LEFT.17; no longer ESP_LEFT_HDR.P$4
- net SR: now also ESP_HDR_RIGHT.18; no longer ESP_LEFT_HDR.P$8
- net S_CURRENT: now also ESP_HDR_LEFT.15; no longer ESP_LEFT_HDR.P$6

Commit message: fixed trace widths of lamp mos and current sensor power traces
Parts:
- added TP1, TP4, TP5: TPB1,27, testpad:TPB1,27
- RTON: value 1.5M -> 781.25k
Connections:
- removed net N$6: C2.1, COUT1.1, COUT2.1, COUT3.1, COUT4.1, R1.2, REG.AGND, REG.PGND, REG.PGND_2, REG.PGND_3, REG.PGND_4
- removed net SPLED_GND: J5.1
- net +5V: now also TP1.TP
- net 3V3: now also TP5.TP
- net GND: now also C2.1, COUT1.1, COUT2.1, COUT3.1, COUT4.1, R1.2, REG.AGND, REG.PGND, REG.PGND_2, REG.PGND_3, REG.PGND_4, TP4.TP
- net PLED_GND: now also J5.1

Commit message: fixed GND labels for individual ports and FETs, rerouted. Fixed GND thickness in MOS sides, Put labels, Combined overhead and primary esp pin nets
Connections:
- removed net D0_GND: R102.1, R105.1, R72.1, R75.1, R78.1, R81.1, R84.1
- removed net D1_GND: R108.1, R111.1, R87.1, R90.1, R93.1, R96.1, R99.1
- removed net D2_GND: R114.1, R117.1, R120.1, R123.1, R126.1, R129.1, R132.1
- removed net OA: R43.2, R44.2
- removed net OGF: R46.2, R47.2
- removed net OGL: R49.2, R50.2
- removed net OGR: R52.2, R53.2
- removed net OLED_GND: J4.1, R42.1, R45.1, R48.1, R51.1, R54.1
- removed net OR: R40.2, R41.2
- removed net PLED_GND: J2.1, J5.1, R10.1, R14.1, R18.1, R25.1, R57.1, R60.1, R63.1, R66.1, R69.1, R7.1
- removed net SLED_GND: J3.1, R21.1, R27.1, R30.1, R36.1, R39.1
- net GND: now also J2.1, J3.1, J4.1, J5.1, R10.1, R102.1, R105.1, R108.1, R111.1, R114.1, R117.1, R120.1, R123.1, R126.1, R129.1, R132.1, R14.1, R18.1, R21.1, R25.1, R27.1, R30.1, R36.1, R39.1, R42.1, R45.1, R48.1, R51.1, R54.1, R57.1, R60.1, R63.1, R66.1, R69.1, R7.1, R72.1, R75.1, R78.1, R81.1, R84.1, R87.1, R90.1, R93.1, R96.1, R99.1
- net PA: now also R43.2, R44.2
- net PGF: now also R46.2, R47.2
- net PGL: now also R49.2, R50.2
- net PGR: now also R52.2, R53.2
- net PR: now also R40.2, R41.2

Commit message: finished v1.1 board and schematic design with Instrumentation amplifier and shunt
Parts:
- removed CB1, CB10, CB11, CB12, CB13, CB14, CB15, CB16, CB17, CB18, CB19, CB2, CB20, CB21, CB22, CB23, CB24, CB25, CB26, CB27, CB28, CB29, CB3, CB30, CB31, CB32, CB33, CB34, CB35, CB36, CB37, CB38, CB39, CB4, CB40, CB5, CB6, CB7, CB8, CB9: 100nF, OPL_Capacitor:CERAMIC-1NF-50V-5%-C0G(0603)
- removed OA_CS, OGF_CS, OGL_CS, OGR_CS, OR_CS, PA_CS, PGF_CS, PGL_CS, PGR_CS, PR_CS, SA_CS, SGF_CS, SGL_CS, SGR_CS, SPA_CS, SPGF_CS, SPGL_CS, SPGR_CS, SPR_CS, SR_CS: ACS723LLCTR-10AU-T, ACS723LLCTR-10AU-T:ACS723LLCTR-10AU-T
- added 3V1, 3V10, 3V11, 3V12, 3V13, 3V14, 3V15, 3V16, 3V17, 3V18, 3V19, 3V2, 3V21, 3V3, 3V4, 3V5, 3V6, 3V7, 3V8, 3V9: MCP40D17T-503E/LT, MCP40D17T-503E_LT:MCP40D17T-503E/LT
- added CEN1, CEN10, CEN11, CEN12, CEN13, CEN14, CEN15, CEN16, CEN17, CEN18, CEN19, CEN2, CEN20, CEN3, CEN4, CEN5, CEN6, CEN7, CEN8, CEN9: 100nF, OPL_Capacitor:CERAMIC-1NF-50V-5%-C0G(0603)
- added R133, R134, R135, R136, R137, R138, R139, R140, R141, R142, R143, R144, R145, R146, R147, R148, R149, R171, R32, R33: CR-02JL6----1K, CR-02JL6----1K:CR-02JL6----1K
- added R150, R151, R152, R153, R154, R155, R156, R157, R158, R159, R160, R161, R162, R163, R164, R165, R166, R167, R168, R172: 1m, RLC16-R100JTP - 100mOhm:RLC16-R100JTP
- added U1, U10, U11, U12, U13, U14, U15, U16, U17, U18, U19, U20, U21, U22, U23, U24, U25, U26, U27, U28: INA332AIDGKR, INA332AIDGKR:INA332AIDGKR
Connections:
- removed net OA_IP-: OA_CS.IP-, Q13.D
- removed net OGF_IP-: OGF_CS.IP-, Q14.D
- removed net OGL_IP-: OGL_CS.IP-, Q15.D
- removed net OGR_IP-: OGR_CS.IP-, Q16.D
- removed net OR_IP-: OR_CS.IP-, Q12.D
- removed net PA_IP-: PA_CS.IP-, Q2.D
- removed net PGF_IP-: PGF_CS.IP-, Q3.D
- removed net PGL_IP-: PGL_CS.IP-, Q4.D
- removed net PGR_IP-: PGR_CS.IP-, Q5.D
- removed net PR_IP-: PR_CS.IP-, Q1.D
- removed net SA_IP-: Q8.D, SA_CS.IP-
- removed net SGF_IP-: Q9.D, SGF_CS.IP-
- removed net SGL_IP-: Q10.D, SGL_CS.IP-
- removed net SGR_IP-: Q11.D, SGR_CS.IP-
- removed net SPA_IP-: Q18.D, SPA_CS.IP-
- removed net SPGF_IP-: Q19.D, SPGF_CS.IP-
- removed net SPGL_IP-: Q20.D, SPGL_CS.IP-
- removed net SPGR_IP-: Q21.D, SPGR_CS.IP-
- removed net SPR_IP-: Q17.D, SPR_CS.IP-
- removed net SR_IP-: Q7.D, SR_CS.IP-
- new net N$10: 3V2.B, R33.1, U10.RG
- new net N$11: R33.2, U10.REF
- new net N$12: 3V3.B, R133.1, U11.RG
- new net N$13: R171.2, U19.REF
- new net N$14: R133.2, U11.REF
- new net N$16: 3V4.B, R134.1, U12.RG
- new net N$17: R134.2, U12.REF
- new net N$19: 3V5.B, R135.1, U13.RG
- new net N$20: R135.2, U13.REF
- new net N$22: 3V6.B, R136.1, U14.RG
- new net N$23: R136.2, U14.REF
- new net N$25: 3V7.B, R137.1, U15.RG
- new net N$26: R137.2, U15.REF
- new net N$28: 3V8.B, R138.1, U16.RG
- new net N$29: R138.2, U16.REF
- new net N$30: 3V9.B, R139.1, U17.RG
- new net N$31: R139.2, U17.REF
- new net N$32: 3V10.B, R140.1, U18.RG
- new net N$33: R140.2, U18.REF
- new net N$34: 3V11.B, R141.1, U20.RG
- new net N$35: R141.2, U20.REF
- new net N$36: 3V12.B, R142.1, U21.RG
- new net N$37: R142.2, U21.REF
- new net N$38: 3V13.B, R143.1, U22.RG
- new net N$39: R143.2, U22.REF
- new net N$4: 3V21.B, R171.1, U19.RG
- new net N$40: 3V14.B, R144.1, U23.RG
- new net N$41: R144.2, U23.REF
- new net N$42: 3V15.B, R145.1, U24.RG
- new net N$43: R145.2, U24.REF
- new net N$44: 3V16.B, R146.1, U25.RG
- new net N$45: R146.2, U25.REF
- new net N$46: 3V17.B, R147.1, U26.RG
- new net N$47: R147.2, U26.REF
- new net N$48: 3V18.B, R148.1, U27.RG
- new net N$49: R148.2, U27.REF
- new net N$5: 3V1.B, R32.1, U1.RG
- new net N$50: 3V19.B, R149.1, U28.RG
- new net N$51: R149.2, U28.REF
- new net N$6: R32.2, U1.REF
- new net OA++: Q13.S, R165.2, U26.VIN+
- new net OGF++: Q14.S, R166.2, U14.VIN+
- new net OGL++: Q15.S, R167.2, U27.VIN+
- new net OGR++: Q16.S, R168.2, U15.VIN+
- new net OR++: Q12.S, R164.2, U13.VIN+
- new net PA++: Q2.S, R150.2, U21.VIN+
- new net PGF++: Q3.S, R151.2, U1.VIN+
- new net PGL++: Q4.S, R152.2, U22.VIN+
- new net PGR++: Q5.S, R153.2, U10.VIN+
- new net PR++: Q1.S, R172.2, U19.VIN+
- new net SA++: Q8.S, R155.2, U11.VIN+
- new net SGF++: Q9.S, R156.2, U24.VIN+
- new net SGL++: Q10.S, R157.2, U12.VIN+
- new net SGR++: Q11.S, R158.2, U25.VIN+
- new net SPA++: Q18.S, R160.2, U16.VIN+
- new net SPGF++: Q19.S, R161.2, U18.VIN+
- new net SPGL++: Q20.S, R162.2, U17.VIN+
- new net SPGR++: Q21.S, R163.2, U20.VIN+
- new net SPR++: Q17.S, R159.2, U28.VIN+
- new net SR++: Q7.S, R154.2, U23.VIN+
- net +5V: now also CEN1.2, CEN10.2, CEN11.2, CEN12.2, CEN13.2, CEN14.2, CEN15.2, CEN16.2, CEN17.2, CEN18.2, CEN19.2, CEN2.2, CEN20.2, CEN3.2, CEN4.2, CEN5.2, CEN6.2, CEN7.2, CEN8.2, CEN9.2, U1.SD, U1.V+, U10.SD, U10.V+, U11.SD, U11.V+, U12.SD, U12.V+, U13.SD, U13.V+, U14.SD, U14.V+, U15.SD, U15.V+, U16.SD, U16.V+, U17.SD, U17.V+, U18.SD, U18.V+, U19.SD, U19.V+, U20.SD, U20.V+, U21.SD, U21.V+, U22.SD, U22.V+, U23.SD, U23.V+, U24.SD, U24.V+, U25.SD, U25.V+, U26.SD, U26.V+, U27.SD, U27.V+, U28.SD, U28.V+; no longer CB1.2, CB11.2, CB13.2, CB15.2, CB17.2, CB19.2, CB21.2, CB23.2, CB25.2, CB27.2, CB29.2, CB3.2, CB31.2, CB33.2, CB35.2, CB37.2, CB39.2, CB5.2, CB7.2, CB9.2, OA_CS.BW_SEL, OA_CS.VCC, OGF_CS.BW_SEL, OGF_CS.VCC, OGL_CS.BW_SEL, OGL_CS.VCC, OGR_CS.BW_SEL, OGR_CS.VCC, OR_CS.BW_SEL, OR_CS.VCC, PA_CS.BW_SEL, PA_CS.VCC, PGF_CS.BW_SEL, PGF_CS.VCC, PGL_CS.BW_SEL, PGL_CS.VCC, PGR_CS.BW_SEL, PGR_CS.VCC, PR_CS.BW_SEL, PR_CS.VCC, SA_CS.BW_SEL, SA_CS.VCC, SGF_CS.BW_SEL, SGF_CS.VCC, SGL_CS.BW_SEL, SGL_CS.VCC, SGR_CS.BW_SEL, SGR_CS.VCC, SPA_CS.BW_SEL, SPA_CS.VCC, SPGF_CS.BW_SEL, SPGF_CS.VCC, SPGL_CS.BW_SEL, SPGL_CS.VCC, SPGR_CS.BW_SEL, SPGR_CS.VCC, SPR_CS.BW_SEL, SPR_CS.VCC, SR_CS.BW_SEL, SR_CS.VCC
- net 3V3: now also 3V1.VDD, 3V10.VDD, 3V11.VDD, 3V12.VDD, 3V13.VDD, 3V14.VDD, 3V15.VDD, 3V16.VDD, 3V17.VDD, 3V18.VDD, 3V19.VDD, 3V2.VDD, 3V21.VDD, 3V3.VDD, 3V4.VDD, 3V5.VDD, 3V6.VDD, 3V7.VDD, 3V8.VDD, 3V9.VDD
- net GND: now also 3V1.VSS, 3V10.VSS, 3V11.VSS, 3V12.VSS, 3V13.VSS, 3V14.VSS, 3V15.VSS, 3V16.VSS, 3V17.VSS, 3V18.VSS, 3V19.VSS, 3V2.VSS, 3V21.VSS, 3V3.VSS, 3V4.VSS, 3V5.VSS, 3V6.VSS, 3V7.VSS, 3V8.VSS, 3V9.VSS, CEN1.1, CEN11.1, CEN12.1, CEN13.1, CEN14.1, CEN15.1, CEN16.1, CEN17.1, CEN18.1, CEN19.1, CEN2.1, CEN20.1, CEN3.1, CEN4.1, CEN5.1, CEN6.1, CEN7.1, CEN8.1, CEN9.1, U1.V-, U10.V-, U11.V-, U12.V-, U13.V-, U14.V-, U15.V-, U16.V-, U17.V-, U18.V-, U19.V-, U20.V-, U21.V-, U22.V-, U23.V-, U24.V-, U25.V-, U26.V-, U27.V-, U28.V-; no longer CB1.1, CB10.1, CB11.1, CB12.1, CB13.1, CB14.1, CB15.1, CB16.1, CB17.1, CB18.1, CB19.1, CB2.1, CB20.1, CB21.1, CB22.1, CB23.1, CB24.1, CB25.1, CB26.1, CB27.1, CB28.1, CB29.1, CB3.1, CB30.1, CB31.1, CB32.1, CB33.1, CB34.1, CB35.1, CB36.1, CB37.1, CB38.1, CB39.1, CB4.1, CB40.1, CB5.1, CB6.1, CB7.1, CB8.1, CB9.1, OA_CS.GND, OGF_CS.GND, OGL_CS.GND, OGR_CS.GND, OR_CS.GND, PA_CS.GND, PGF_CS.GND, PGL_CS.GND, PGR_CS.GND, PR_CS.GND, SA_CS.GND, SGF_CS.GND, SGL_CS.GND, SGR_CS.GND, SPA_CS.GND, SPGF_CS.GND, SPGL_CS.GND, SPGR_CS.GND, SPR_CS.GND, SR_CS.GND
- net I_OA: now also 3V17.W, U26.VOUT; no longer CB16.2, OA_CS.VIOUT
- net I_OGF: now also 3V6.W, U14.VOUT; no longer CB18.2, OGF_CS.VIOUT
- net I_OGL: now also 3V18.W, U27.VOUT; no longer CB20.2, OGL_CS.VIOUT
- net I_OGR: now also 3V7.W, U15.VOUT; no longer CB22.2, OGR_CS.VIOUT
- net I_OR: now also 3V5.W, U13.VOUT; no longer CB14.2, OR_CS.VIOUT
- net I_PA: now also 3V12.W, U21.VOUT; no longer CB24.2, PA_CS.VIOUT
- net I_PGF: now also 3V1.W, U1.VOUT; no longer CB36.2, PGF_CS.VIOUT
- net I_PGL: now also 3V13.W, U22.VOUT; no longer CB38.2, PGL_CS.VIOUT
- net I_PGR: now also 3V2.W, U10.VOUT; no longer CB40.2, PGR_CS.VIOUT
- net I_PR: now also 3V21.W, U19.VOUT; no longer CB12.2, PR_CS.VIOUT
- net I_SA: now also 3V3.W, U11.VOUT; no longer CB6.2, SA_CS.VIOUT
- net I_SGF: now also 3V15.W, U24.VOUT; no longer CB8.2, SGF_CS.VIOUT
- net I_SGL: now also 3V4.W, U12.VOUT; no longer CB2.2, SGL_CS.VIOUT
- net I_SGR: now also 3V16.W, U25.VOUT; no longer CB10.2, SGR_CS.VIOUT
- net I_SPA: now also 3V8.W, U16.VOUT; no longer CB28.2, SPA_CS.VIOUT
- net I_SPGF: now also 3V10.W, U18.VOUT; no longer CB30.2, SPGF_CS.VIOUT
- net I_SPGL: now also 3V9.W, U17.VOUT; no longer CB32.2, SPGL_CS.VIOUT
- net I_SPGR: now also 3V11.W, U20.VOUT; no longer CB34.2, SPGR_CS.VIOUT
- net I_SPR: now also 3V19.W, U28.VOUT; no longer CB26.2, SPR_CS.VIOUT
- net I_SR: now also 3V14.W, U23.VOUT; no longer CB4.2, SR_CS.VIOUT
- net OA+: now also R165.1, U26.VIN-; no longer Q13.S
- net OGF+: now also R166.1, U14.VIN-; no longer Q14.S
- net OGL+: now also R167.1, U27.VIN-; no longer Q15.S
- net OGR+: now also R168.1, U15.VIN-; no longer Q16.S
- net OR+: now also R164.1, U13.VIN-; no longer Q12.S
- net PA+: now also R150.1, U21.VIN-; no longer Q2.S
- net PGF+: now also R151.1, U1.VIN-; no longer Q3.S
- net PGL+: now also R152.1, U22.VIN-; no longer Q4.S
- net PGR+: now also R153.1, U10.VIN-; no longer Q5.S
- net PR+: now also R172.1, U19.VIN-; no longer Q1.S
- net SA+: now also R155.1, U11.VIN-; no longer Q8.S
- net SCL: now also 3V1.SCL, 3V10.SCL, 3V11.SCL, 3V12.SCL, 3V13.SCL, 3V14.SCL, 3V15.SCL, 3V16.SCL, 3V17.SCL, 3V18.SCL, 3V19.SCL, 3V2.SCL, 3V21.SCL, 3V3.SCL, 3V4.SCL, 3V5.SCL, 3V6.SCL, 3V7.SCL, 3V8.SCL, 3V9.SCL
- net SDA: now also 3V1.SDA, 3V10.SDA, 3V11.SDA, 3V12.SDA, 3V13.SDA, 3V14.SDA, 3V15.SDA, 3V16.SDA, 3V17.SDA, 3V18.SDA, 3V19.SDA, 3V2.SDA, 3V21.SDA, 3V3.SDA, 3V4.SDA, 3V5.SDA, 3V6.SDA, 3V7.SDA, 3V8.SDA, 3V9.SDA
- net SGF+: now also R156.1, U24.VIN-; no longer Q9.S
- net SGL+: now also R157.1, U12.VIN-; no longer Q10.S
- net SGR+: now also R158.1, U25.VIN-; no longer Q11.S
- net SPA+: now also R160.1, U16.VIN-; no longer Q18.S
- net SPGF+: now also R161.1, U18.VIN-; no longer Q19.S
- net SPGL+: now also R162.1, U17.VIN-; no longer Q20.S
- net SPGR+: now also R163.1, U20.VIN-; no longer Q21.S
- net SPR+: now also R159.1, U28.VIN-; no longer Q17.S
- net SR+: now also R154.1, U23.VIN-; no longer Q7.S
- net VIN: now also Q1.D, Q10.D, Q11.D, Q12.D, Q13.D, Q14.D, Q15.D, Q16.D, Q17.D, Q18.D, Q19.D, Q2.D, Q20.D, Q21.D, Q3.D, Q4.D, Q5.D, Q7.D, Q8.D, Q9.D; no longer OA_CS.IP+, OGF_CS.IP+, OGL_CS.IP+, OGR_CS.IP+, OR_CS.IP+, PA_CS.IP+, PGF_CS.IP+, PGL_CS.IP+, PGR_CS.IP+, PR_CS.IP+, SA_CS.IP+, SGF_CS.IP+, SGL_CS.IP+, SGR_CS.IP+, SPA_CS.IP+, SPGF_CS.IP+, SPGL_CS.IP+, SPGR_CS.IP+, SPR_CS.IP+, SR_CS.IP+
Other:
- note added: "Overhead"
- note added: "Primary"
- note added: "Secondary"
- note added: "Spare"
- note removed: "Overhead Lamp FETs and Port"
- note removed: "Primary Lamp FETs and Port"
- note removed: "Secondary Lamp FETs and Port"
- note removed: "Spare Lamp FETs and Port"
- moved on the sheet: C2, C3, C4, C5, CB, CEN, CIN1, CIN2, CIN3, COUT1, COUT2, COUT3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
